File: hardware_machine_lock/_autosave-raspi_nfc_machine_lock.sch (KiCad schematic (older format))
At the start: 90 parts, among them J101 Raspberry_Pi_2_3, J102 Conn_01x04, J103 Screw_Terminal_01x02, J104 Screw_Terminal_01x02, J105 Conn_01x08, J106 Screw_Terminal_01x03, J107 Screw_Terminal_01x02, J108 Screw_Terminal_01x02, J113 BUZZER, K101 G5Q-1A, Q101 MMBT3904, Q103 MMBT3904, U101 74HC14, U102 LM2596S-5.0, U105 ADS1115IDGS

Commit message: Update KiCad version
Parts:
- gave numbers to parts that had none: 2
Changed lines of the file:
@@
 NoConn ~ 8100 7350
 $Comp
-L Connector:Screw_Terminal_01x02 J?
+L Connector:Screw_Terminal_01x02 J109
 U 1 1 611A5445
 P 1450 9350
-F 0 "J?" H 1368 9025 50  0000 C CNN
+F 0 "J109" H 1368 9025 50  0000 C CNN
 F 1 "Screw_Terminal_01x02" V 1600 9250 50  0000 C CNN
 F 2 "TerminalBlock_Phoenix:TerminalBlock_Phoenix_MPT-0,5-2-2.54_1x02_P2.54mm_Horizontal" H 1450 9350 50  0001 C CNN
@@
 External CT
 $Comp
-L PSK-10D-12:PSK-10D-12 PS?
+L PSK-10D-12:PSK-10D-12 PS101
 U 1 1 6177C23D
 P 2800 3350
-F 0 "PS?" H 2800 3717 50  0000 C CNN
+F 0 "PS101" H 2800 3717 50  0000 C CNN
 F 1 "PSK-10D-12" H 2800 3626 50  0000 C CNN
 F 2 "CONV_PSK-10D-12" H 2800 3350 50  0001 L BNN
